File: blocks/nRF54L.kicad_blocks/nRF54L15-CAAA_Reference_Design.kicad_block/nRF54L15-CAAA_Reference_Design.kicad_sch (KiCad schematic)
At the start: 16 parts, among them U1 nRF54L15-CAXX, Y1 32MHz

Commit message: Updates to move to auto-generated footprints
Parts:
- U1: footprint nordic-lib-kicad-nrf54:BGA-47_7x7_2.451x2.245mm -> nordic-lib-kicad-nrf54l:BGA-47_7x7_2.451x2.245mm
Changed lines of the file:
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@@
 			)
 		)
-		(property "Footprint" "nordic-lib-kicad-nrf54:BGA-47_7x7_2.451x2.245mm"
+		(property "Footprint" "nordic-lib-kicad-nrf54l:BGA-47_7x7_2.451x2.245mm"
 			(at 140.97 109.22 0)
 			(effects
