File: libmanagement/libmanagement.kicad_sch (KiCad schematic)
At the start: 0 parts

Commit message: Assign 32MHz crystal footprint and LCSC part
Parts:
- added C1: 10uF, Capacitor_SMD:C_0402_1005Metric, symbol Device:C_Small
- added C10: 1.2pF, symbol Device:C_Small
- added C11: 1.5pF, symbol Device:C_Small
- added C12: NC, symbol Device:C_Small
- added C2, C3, C4: 1uF, symbol Device:C_Small
- added C5, C9: 4.7uF, Capacitor_SMD:C_0402_1005Metric, symbol Device:C_Small
- added C6, C8: 2.2uF, symbol Device:C_Small
- added C7: 1pF, symbol Device:C_Small
- added FB1: 120R @ 100MHz, symbol Device:FerriteBead_Small
- added L1: 4.7uH, Inductor_SMD:L_0603_1608Metric, symbol Device:L_Small
- added L2: 1nH, symbol Device:L_Small
- added L3: 3.6nH, symbol Device:L_Small
- added L4: 4.7nH, symbol Device:L_Small
- added L5: 3.3nH, symbol Device:L_Small
- added R1: 200R, Resistor_SMD:R_0201_0603Metric, symbol Device:R_Small_US
- added R2: 2R2, Resistor_SMD:R_0603_1608Metric, symbol Device:R_Small_US
- added U1: nRF54LM20A-QGXX, nordic-lib-kicad-nrf54l:QFN-52-1EP_6x6mm_P0.4mm_EP4.7x4.7mm_ThermalVias, symbol nordic-lib-kicad-nrf54l:nRF54LM20A-QGXX
- added Y1: 32.768KHz, Crystal:Crystal_SMD_2012-2Pin_2.0x1.2mm, symbol Device:Crystal_Small
- added Y2: 32MHz, Crystal:Crystal_SMD_2016-4Pin_2.0x1.6mm, symbol Device:Crystal_GND24_Small
Connections:
- new net: C5.1, FB1.1, L1.2, U1.44 (DECD)
- new net: C6.1, C7.1, FB1.2, L2.2, U1.46 (DECA)
- new net: C7.2, L2.1, U1.36 (DECRF)
- new net: C1.1, C2.1, C3.1, C4.1, U1.42 (VDD), U1.51 (VDD), U1.6 (VDD)
- new net: C8.1, U1.18 (DECUSB)
- new net: L3.1, U1.34 (ANT)
- new net: C10.1, L3.2, L4.1
- new net: C11.1, L4.2, L5.1
- new net: C12.1, L5.2
- new net: U1.49 (P1.21), Y1.1
- new net: U1.48 (P1.20), Y1.2
- new net: C9.1, R2.2, U1.17 (VBUS)
- new net: R1.1, U1.21 (TXRTUNE)
- new net: U1.37 (XC1), Y2.1
- new net: U1.38 (XC2), Y2.3
- new net: L1.1, U1.43 (DCC)
- new net GND: C1.2, C10.2, C11.2, C12.2, C2.2, C3.2, C4.2, C5.2, C6.2, C8.2, C9.2, R1.2, U1.35 (VSS), U1.45 (VSS), U1.53 (VSS), Y2.2, Y2.4
- new net VBUS: R2.1
