File: libmanagement/libmanagement.kicad_sch (KiCad schematic)
At the start: 0 parts

Commit message: updates for ref design test
Parts:
- added C1: 10uF, Capacitor_SMD:C_0402_1005Metric, symbol Device:C_Small
- added C10, C5: 2.2uF, Capacitor_SMD:C_0201_0603Metric, symbol Device:C_Small
- added C11: 0.3pF, Capacitor_SMD:C_0201_0603Metric, symbol Device:C_Small
- added C12: 10nF, Capacitor_SMD:C_0201_0603Metric, symbol Device:C_Small
- added C13: 2.2nF, Capacitor_SMD:C_0201_0603Metric, symbol Device:C_Small
- added C2, C3, C6, C8: 100nF, Capacitor_SMD:C_0201_0603Metric, symbol Device:C_Small
- added C4: 3.9pF, Capacitor_SMD:C_0201_0603Metric, symbol Device:C_Small
- added C7: 1.5pF, Capacitor_SMD:C_0201_0603Metric, symbol Device:C_Small
- added C9: 2.0pF, Capacitor_SMD:C_0201_0603Metric, symbol Device:C_Small
- added FB1: 100R@100MHz, Inductor_SMD:L_0201_0603Metric, symbol Device:FerriteBead_Small
- added L1: 4.7uH, Inductor_SMD:L_0603_1608Metric, symbol Device:L_Small
- added L2: 2.7nH, Inductor_SMD:L_0201_0603Metric, symbol Device:L_Small
- added L3, L4: 3.5nH, Inductor_SMD:L_0201_0603Metric, symbol Device:L_Small
- added R1: 1kR, Resistor_SMD:R_0201_0603Metric, symbol Device:R_Small_US
- added U1: nRF54L15-QFXX, Package_DFN_QFN:QFN-48-1EP_6x6mm_P0.4mm_EP4.6x4.6mm_ThermalVias, symbol nordic-lib-kicad-nrf54l:nRF54L15-QFXX
Connections:
- new net: C4.1, R1.1, U1.30 (~{RESET})
- new net: C10.1, C12.1, C13.1, FB1.1, U1.33 (DECRF), U1.43 (DECA)
- new net: C5.1, FB1.2, L1.1, U1.45 (DECD)
- new net: C1.1, C2.1, C3.1, C6.1, C8.1, U1.10 (VDD), U1.22 (VDD), U1.36 (VDD), U1.47 (VDD), U1.48 (VDD)
- new net: C9.1, L3.2, L4.1
- new net: C7.1, L2.2, L3.1
- new net: L2.1, U1.31 (ANT)
- new net: L1.2, U1.46 (DCC)
- new net ANT: C11.1, L4.2
- new net GND: C1.2, C10.2, C11.2, C12.2, C13.2, C2.2, C3.2, C4.2, C5.2, C6.2, C7.2, C8.2, C9.2, U1.32 (VSS_PA), U1.44 (VSS), U1.49 (VSS)
- new net ~{RESET}: R1.2
