File: libmanagement/libmanagement.kicad_pcb (KiCad board)
At the start: 2 copper layers, 16 parts, among them U1 nPM1100-CAXX, U10 nRF7001-QFXX, U11 nRF7002-QFXX, U12 nRF9151-LAXX, U13 nRF9160-SIXX, U14 nRF9161-SIXX, U2 nPM1300-CAXX, U3 nPM2100-CAXX, U4 nPM6001-CAXX, U5 nPM1100-QDXX, U6 nPM1300-QEXX, U7 nPM2100-QEXX, U8 nRF7002-CEXX, U9 nRF7000-QFXX

Commit message: updates for ref design test
Parts:
- removed REF**: BC15C-LGA-36_6x12.4mm, PCM_nordic-lib-kicad-nrf54-modules:BC15C-LGA-36_6x12.4mm
- removed REF**: Nordic_nRF9151-LAxx_LGA-80-33EP_12.1x11.1mm_P0.5mm, Package_LGA:Nordic_nRF9151-LAxx_LGA-80-33EP_12.1x11.1mm_P0.5mm
- removed the U1 at (141.7, 107.8)
- removed U10: nRF7001-QFXX, Package_DFN_QFN:QFN-48-1EP_6x6mm_P0.4mm_EP4.6x4.6mm_ThermalVias
- removed U11: nRF7002-QFXX, Package_DFN_QFN:QFN-48-1EP_6x6mm_P0.4mm_EP4.6x4.6mm_ThermalVias
- removed U12: nRF9151-LAXX, PCM_nordic-lib-kicad-nrf9:LGA_9151_12.1x11.1mm
- removed U13: nRF9160-SIXX, PCM_nordic-lib-kicad-nrf9:LGA_9160_16.0x10.5mm
- removed U14: nRF9161-SIXX, PCM_nordic-lib-kicad-nrf9:LGA_9161_16.0x10.5mm
- removed U2: nPM1300-CAXX, PCM_nordic-lib-kicad-npm:BGA-35_7x5_3.077x2.3775mm
- removed U3: nPM2100-CAXX, PCM_nordic-lib-kicad-npm:BGA-16_4x4_1.9175x1.8975mm
- removed U4: nPM6001-CAXX, PCM_nordic-lib-kicad-npm:BGA-45_5x9_2.175x3.635mm
- removed U5: nPM1100-QDXX, Package_DFN_QFN:QFN-24-1EP_4x4mm_P0.5mm_EP2.6x2.6mm_ThermalVias
- removed U6: nPM1300-QEXX, Package_DFN_QFN:QFN-32-1EP_5x5mm_P0.5mm_EP3.6x3.6mm_ThermalVias
- removed U7: nPM2100-QEXX, Package_DFN_QFN:UQFN-16-1EP_4x4mm_P0.65mm_EP2.6x2.6mm_ThermalVias
- removed U8: nRF7002-CEXX, PCM_nordic-lib-kicad-nrf7:BGA-90_10x9_3.7495x3.385mm
- removed U9: nRF7000-QFXX, Package_DFN_QFN:QFN-48-1EP_6x6mm_P0.4mm_EP4.6x4.6mm_ThermalVias
- added C1: 2.2µF, Parts$:CAPC0603X03L_C, F.Cu at (205.0, 137.7)
- added C1: 2.2µF, Parts$:CAPC0603X03L_C, F.Cu at (191.1, 149.7)
- added C1: 10uF, Capacitor_SMD:C_0402_1005Metric, F.Cu at (188.2, 136.7)
- added C10: 100nF, CAPC0603X03L_C:CAPC0603X03L_C, F.Cu at (203.5, 137.7)
- added C10: 100nF, CAPC0603X03L_C:CAPC0603X03L_C, F.Cu at (189.7, 149.7)
- added C10: 2.2uF, Capacitor_SMD:C_0201_0603Metric, F.Cu at (192.5, 135.8)
- added C11: 0.3pF, CAPC0603X03L_C:CAPC0603X03L_C, F.Cu at (199.7, 153.0)
- added C11: 0.3pF, Capacitor_SMD:C_0201_0603Metric, F.Cu at (180.7, 134.8)
- added C11: 0.3pF, CAPC0603X03L_C:CAPC0603X03L_C, F.Cu at (213.6, 141.0)
- added C12: 10nF, CAPC0603X03L_C:CAPC0603X03L_C, F.Cu at (192.0, 149.4)
- added C12: 10nF, Capacitor_SMD:C_0201_0603Metric, F.Cu at (192.1, 137.3)
- added C12: 10nF, CAPC0603X03L_C:CAPC0603X03L_C, F.Cu at (205.9, 137.4)
- added C13: 10nF, Capacitor_SMD:C_0201_0603Metric, F.Cu at (196.3, 140.0)
- added C13: 3.9pF, CAPC0603X03L_C:CAPC0603X03L_C, F.Cu at (196.2, 154.0)
- added C13: 3.9pF, CAPC0603X03L_C:CAPC0603X03L_C, F.Cu at (210.0, 142.0)
- added C2: 100nF, Capacitor_SMD:C_0201_0603Metric, F.Cu at (187.9, 143.3)
- added C2: 2.2µF, Parts$:CAPC0603X03L_C, F.Cu at (192.7, 147.8)
- added C2: 2.2µF, Parts$:CAPC0603X03L_C, F.Cu at (206.5, 135.8)
- added C3: 10µF, Parts$:CAPC1005X04L, F.Cu at (188.5, 148.7)
- added C3: 10µF, Parts$:CAPC1005X04L, F.Cu at (202.4, 136.7)
- added C3: 100nF, Capacitor_SMD:C_0201_0603Metric, F.Cu at (193.7, 145.6)
- added C4: 100nF, CAPC0603X03L_C:CAPC0603X03L_C, F.Cu at (195.6, 150.6)
- added C4: 3.9pF, Capacitor_SMD:C_0201_0603Metric, F.Cu at (178.2, 133.0)
- added C4: 100nF, CAPC0603X03L_C:CAPC0603X03L_C, F.Cu at (209.4, 138.6)
- added C5: 2.2uF, Capacitor_SMD:C_0201_0603Metric, F.Cu at (191.0, 137.7)
- added C5: 2.2nF, Passive:CAPC0603X03L_C, F.Cu at (196.2, 152.4)
- added C5: 2.2nF, Passive:CAPC0603X03L_C, F.Cu at (210.0, 140.4)
- added C6: 100nF, Capacitor_SMD:C_0201_0603Metric, F.Cu at (195.9, 138.6)
- added C6: 1.5pF, CAPC0603X03L_C:CAPC0603X03L_C, F.Cu at (196.2, 152.9)
- added C6: 1.5pF, CAPC0603X03L_C:CAPC0603X03L_C, F.Cu at (210.0, 140.9)
- added C7: 1.5pF, Capacitor_SMD:C_0201_0603Metric, F.Cu at (196.3, 140.7)
- added C7: 100nF, CAPC0603X03L_C:CAPC0603X03L_C, F.Cu at (201.8, 143.3)
- added C7: 100nF, CAPC0603X03L_C:CAPC0603X03L_C, F.Cu at (187.9, 155.3)
- added C8: 100nF, Capacitor_SMD:C_0201_0603Metric, F.Cu at (189.5, 137.7)
- added C8: 100nF, CAPC0603X03L_C:CAPC0603X03L_C, F.Cu at (207.5, 145.6)
- added C8: 100nF, CAPC0603X03L_C:CAPC0603X03L_C, F.Cu at (193.7, 157.6)
- added C9: 2.0pF, CAPC0603X03L_C:CAPC0603X03L_C, F.Cu at (198.1, 153.7)
- added C9: 2.0pF, Capacitor_SMD:C_0201_0603Metric, F.Cu at (180.7, 131.2)
- added C9: 2.0pF, CAPC0603X03L_C:CAPC0603X03L_C, F.Cu at (211.9, 141.7)
- added FB1: 120R/0.2A, INDC0603X03L_C:INDC0603X03L_C, F.Cu at (192.0, 147.8)
- added FB1: 120R/0.2A, INDC0603X03L_C:INDC0603X03L_C, F.Cu at (205.9, 135.8)
- added FB1: 100R@100MHz, Inductor_SMD:L_0201_0603Metric, F.Cu at (191.8, 135.8)
- added L1: 4.7µH, 0603:INDC1608X06L, F.Cu at (204.0, 136.4)
- added L1: 4.7µH, 0603:INDC1608X06L, F.Cu at (190.1, 148.4)
- added L1: 4.7uH, Inductor_SMD:L_0603_1608Metric, F.Cu at (190.2, 136.4)
- added L2: 2.7nH, Inductor_SMD:L_0201_0603Metric, F.Cu at (196.3, 141.4)
- added L2: 2.7nH, Passive:INDC0603X03L_C, F.Cu at (210.0, 141.4)
- added L2: 2.7nH, Passive:INDC0603X03L_C, F.Cu at (196.2, 153.4)
- added L3: 3.5nH, INDC0603X03L_C:INDC0603X03L_C, F.Cu at (211.1, 141.4)
- added L3: 3.5nH, INDC0603X03L_C:INDC0603X03L_C, F.Cu at (197.3, 153.4)
- added L3: 3.5nH, Inductor_SMD:L_0201_0603Metric, F.Cu at (183.1, 133.0)
- added L4: 3.5nH, INDC0603X03L_C:INDC0603X03L_C, F.Cu at (198.9, 153.4)
- added L4: 3.5nH, INDC0603X03L_C:INDC0603X03L_C, F.Cu at (212.8, 141.4)
- added L4: 3.5nH, Inductor_SMD:L_0201_0603Metric, F.Cu at (183.1, 134.8)
- added R1: 1k, RESC0603X03L_C:RESC0603X03L_C, F.Cu at (210.5, 142.6)
- added R1: 1kR, Resistor_SMD:R_0201_0603Metric, F.Cu at (183.1, 136.5)
- added R1: 1k, RESC0603X03L_C:RESC0603X03L_C, F.Cu at (196.7, 154.6)
- added U1: nRF54L15-QFAA, Misc:QFN40P600X600X90-48N, F.Cu at (205.8, 141.6)
- added U1: nRF54L15-QFXX, Package_DFN_QFN:QFN-48-1EP_6x6mm_P0.4mm_EP4.6x4.6mm_ThermalVias, F.Cu at (192.0, 141.6)
- added U1: nRF54L15-QFAA, Misc:QFN40P600X600X90-48N, F.Cu at (192.0, 153.6)
- added X1: 32.768kHz, Parts$:XTAL_2012, F.Cu at (201.0, 139.4)
- added X1: 32.768kHz, Parts$:XTAL_2012, F.Cu at (187.2, 151.4)
- added X2: 32MHz, Parts$:BT-XTAL_2016, F.Cu at (197.4, 149.9)
- added X2: 32MHz, Parts$:BT-XTAL_2016, F.Cu at (211.2, 137.9)
- added Y1: 32MHz, Crystal:Crystal_SMD_2016-4Pin_2.0x1.6mm, F.Cu at (197.6, 137.9)
